Commit message: converted line_follower_robot urdf file to xacro and changed launch files respectively

File: gazebo_ws/src/simple_robot_car/urdf/simple_robot_car.urdf (robot description, URDF)
Before this commit: robot simple_robot_car, 5 links, 4 joints
Joints:
- joint FR_wheel_joint: origin xyz=0.02286 0.02413 -0.0127 rpy=0 0 0 -> xyz=0.0 0.0 0.0 rpy=0 0 0
