Commit message: cleaned up workspace and launch files, issues with STL meashes persists in gazebo

File: gazebo_ws/src/line_follower_robot/urdf/line_follower_robot.urdf.xacro (robot description, xacro)
@@ -9,4 +9,13 @@
   <xacro:property name="castor_base_mesh" value="package://line_follower_robot/meshes/castor_base_link.STL"/>
   <xacro:property name="castor_wheel_mesh" value="package://line_follower_robot/meshes/castor_wheel.STL"/>
+  <!-- ========================= -->
+  <!-- world link -->
+  <!-- ========================= -->
+  <link name="world"/>
+  <joint name="world_joint" type="fixed">
+    <parent link="world"/>
+    <child link="base_link"/>
+    <origin xyz="0 0 1" rpy="0 0 0"/>
+  </joint>
   <!-- ========================= -->
   <!-- Base link -->
@@ -109,4 +118,15 @@
       </material>
     </visual>
+    <inertial>
+      <origin xyz="0 0 0" rpy="0 0 0"/>
+      <mass value="0.01"/>
+      <inertia ixx="0.00001" ixy="0" ixz="0" iyy="0.00001" iyz="0" izz="0.00001"/>
+    </inertial>
+    <collision>
+     <origin xyz="0 0 0" rpy="0 0 0"/>
+      <geometry>
+        <mesh filename="${castor_wheel_mesh}"/>
+      </geometry>
+    </collision>
   </link>
   <joint name="castor_joint" type="continuous">
@@ -122,4 +142,15 @@
       </geometry>
     </visual>
+    <inertial>
+      <origin xyz="0 0 0" rpy="0 0 0"/>
+      <mass value="0.01"/>
+      <inertia ixx="0.00001" ixy="0" ixz="0" iyy="0.00001" iyz="0" izz="0.00001"/>
+    </inertial>
+    <collision>
+     <origin xyz="0 0 0" rpy="0 0 0"/>
+      <geometry>
+        <mesh filename="${castor_wheel_mesh}"/>
+      </geometry>
+    </collision>
   </link>
   <joint name="castor_wheel_joint" type="continuous">

File: gazebo_ws/src/mobilerobot/urdf/mobilebot.urdf.xacro (robot description, xacro)
@@ -2,3 +2,4 @@
 <robot xmlns:xacro="http://www.ros.org/wiki/xacro" name="mobilebot">
     <xacro:include filename="mobilerobot.xacro" />
+    <xacro:include filename="gazebo_control.xacro" />
 </robot>

File: gazebo_ws/src/mobilerobot/urdf/mobilerobot.xacro (robot description, xacro)
@@ -1,5 +1,5 @@
-<?xml version="1.0"?>
+xml version="1.0"?>
 <robot xmlns:xacro="http://www.ros.org/wiki/xacro" name="mobilebot">
-  <!-- Materials -->
+  <!-- Materials --><?
   <material name="red"><color rgba="1 0 0 1"/></material>
   <material name="green"><color rgba="0 1 0 1"/></material>
