Commit message: cafeteria build file created

File: colcon_ws/src/rviz_tutorial/urdf/camera.xacro (robot description, xacro)
@@ -19,10 +19,10 @@
         <parent link="base_link"/>
         <child link="camera_link"/>
-        <origin xyz="-0.08 0.0 0.15" rpy="0 0 ${pi}"/>
+        <origin xyz="0.08 0.0 0.15" rpy="0 0 0"/>
     </joint>
     <joint name="camera_optical_joint" type="fixed">
         <parent link="camera_link"/>
         <child link="camera_link_optical"/>
-        <origin xyz="-0.08 0 0.15" rpy="${-pi/2} 0 ${pi/2}"/>
+        <origin xyz="0.08 0 0.15" rpy="${-pi/2} 0 ${pi/2}"/>
     </joint>
     <link name="camera_link_optical"></link>

File: colcon_ws/src/rviz_tutorial/urdf/lidar.xacro (robot description, xacro)
@@ -21,5 +21,5 @@
         <child link="laser_frame"/>
         <!-- place wheel at front-right of base (x, y, z) -->
-        <origin xyz="0.08 0.0 0.15"/>
+        <origin xyz="0.0 0.0 0.15"/>
   </joint>
     <gazebo reference="laser_frame">
@@ -38,5 +38,5 @@
                 </scan>
                 <range>
-                    <min>0.3</min>
+                    <min>0.2</min>
                     <max>12</max>
                 </range>

File: colcon_ws/src/rviz_tutorial/urdf/simple_robot_car.xacro (robot description, xacro)
@@ -136,6 +136,6 @@
       </ros>
       <!-- wheel iformation-->
-      <left_joint>body_left_wheel</left_joint>
-      <right_joint>body_right_wheel</right_joint>
+      <left_joint>body_right_wheel</left_joint>
+      <right_joint>body_left_wheel</right_joint>
       <wheel_separation>${wheel_separation}</wheel_separation>
       <wheel_diameter>0.08</wheel_diameter>
