Commit message: slam map error fixed, cartographer not fixed

File: colcon_ws/src/rviz_tutorial/urdf/IMU_link.xacro (robot description, xacro)
@@ -21,19 +21,3 @@
         <origin xyz="-0.08 0.0 0.15" rpy="0 0 0"/>
     </joint>
-    <gazebo reference="imu_link">
-        <material>Gazebo/Red</material>
-        <sensor name="imu_sensor" type="imu">
-            <pose> 0 0 0 0 0 0 </pose>
-            <always_on>true</always_on>
-            <visualize>true</visualize>
-            <update_rate>50</update_rate>
-            <plugin name="Imu_plugin" filename="libgazebo_ros_imu_sensor.so">
-                <ros>
-                    <remapping>~/out:=/imu</remapping>
-                </ros>
-                <output_type>sensor_msgs/msg/imu</output_type>
-                <frame_name>imu_link</frame_name>
-            </plugin>
-        </sensor>
-    </gazebo>
 </robot>

File: colcon_ws/src/rviz_tutorial/urdf/robot.urdf.xacro (robot description, xacro)
@@ -4,4 +4,4 @@
     <xacro:include filename="$(find rviz_tutorial)/urdf/lidar.xacro"/>
     <xacro:include filename="$(find rviz_tutorial)/urdf/camera.xacro"/>
-    <xacro:include filename="$(find rviz_tutorial)/urdf/IMU_link.xacro"/>
+    <!--xacro:include filename="$(find rviz_tutorial)/urdf/IMU_link.xacro"/-->
 </robot>
